File: hardware/2ch-4-20mA/2ch-4-20mA.sch (KiCad schematic (older format))
At the start: 29 parts, among them J1 Conn_01x02, J2 Conn_01x02, J3 Conn_01x07, U1 LMP8640, U2 LMP8640, U3 TEC2-0913

Commit message: Updated PCB with new OSHW logo
Parts:
- G1: footprint BrechtVE_Aesthetics:OSHW-EEVBLOG2_SPFMDBC_SolderMaskTop_5mm -> BrechtVE_Aesthetics:OSHW-Logo_5.7x6mm_SolderMask; symbol BrechtVE_Aesthetics:Symbol_OSHW-EEVBLOG_SPFMDBC_10mm -> BrechtVE_Aesthetics:Symbol_OSHW-Logo_11.4x12mm
- H1, H2, H3, H4: value MountingHole -> M3
Other:
- note removed: "M3 holes"
Changed lines of the file:
@@
 U 1 1 5DD493BC
 P 10100 7050
-F 0 "H1" H 10200 7050 50  0000 L CNN
-F 1 "MountingHole" H 10200 7005 50  0001 L CNN
+F 0 "H1" H 10200 7100 50  0000 L CNN
+F 1 "M3" H 10200 7005 50  0000 L CNN
 F 2 "MountingHole:MountingHole_3.2mm_M3" H 10100 7050 50  0001 C CNN
 F 3 "~" H 10100 7050 50  0001 C CNN
@@
 U 1 1 5DD4988A
 P 10400 7050
-F 0 "H2" H 10500 7050 50  0000 L CNN
-F 1 "MountingHole" H 10500 7005 50  0001 L CNN
+F 0 "H2" H 10500 7100 50  0000 L CNN
+F 1 "M3" H 10500 7005 50  0000 L CNN
 F 2 "MountingHole:MountingHole_3.2mm_M3" H 10400 7050 50  0001 C CNN
 F 3 "~" H 10400 7050 50  0001 C CNN
@@
 U 1 1 5DD49B52
 P 10700 7050
-F 0 "H3" H 10800 7050 50  0000 L CNN
-F 1 "MountingHole" H 10800 7005 50  0001 L CNN
+F 0 "H3" H 10800 7100 50  0000 L CNN
+F 1 "M3" H 10800 7005 50  0000 L CNN
 F 2 "MountingHole:MountingHole_3.2mm_M3" H 10700 7050 50  0001 C CNN
 F 3 "~" H 10700 7050 50  0001 C CNN
@@
 U 1 1 5DD49EB8
 P 11000 7050
-F 0 "H4" H 11100 7050 50  0000 L CNN
-F 1 "MountingHole" H 11100 7005 50  0001 L CNN
+F 0 "H4" H 11100 7100 50  0000 L CNN
+F 1 "M3" H 11100 7005 50  0000 L CNN
 F 2 "MountingHole:MountingHole_3.2mm_M3" H 11000 7050 50  0001 C CNN
 F 3 "~" H 11000 7050 50  0001 C CNN
@@
 Wire Wire Line
 	6450 2900 6500 2900
-Text Notes 9650 7100 0    50   ~ 0
-M3 holes
 $Comp
 L Device:Jumper_NC_Small JP4
@@
 Connection ~ 7650 4350
 $Comp
-L BrechtVE_Aesthetics:Symbol_OSHW-EEVBLOG_SPFMDBC_10mm G1
+L BrechtVE_Aesthetics:Symbol_OSHW-Logo_11.4x12mm G1
 U 1 1 5DDA859B
-P 11000 6350
-F 0 "G1" H 11000 6175 60  0001 C CNN
-F 1 "OSHW-EEVBLOG-SPFMDBC-10mm" H 11000 6525 60  0001 C CNN
-F 2 "BrechtVE_Aesthetics:OSHW-EEVBLOG2_SPFMDBC_SolderMaskTop_5mm" H 11000 6350 50  0001 C CNN
-F 3 "" H 11000 6350 50  0001 C CNN
-	1    11000 6350
+P 10950 6400
+F 0 "G1" H 10950 6225 60  0001 C CNN
+F 1 "OSHW-EEVBLOG-SPFMDBC-10mm" H 10950 6575 60  0001 C CNN
+F 2 "BrechtVE_Aesthetics:OSHW-Logo_5.7x6mm_SolderMask" H 10950 6400 50  0001 C CNN
+F 3 "" H 10950 6400 50  0001 C CNN
+	1    10950 6400
 	1    0    0    -1
 $EndComp
